File: 4in1ESC.kicad_sch (KiCad schematic)
At the start: 53 parts, among them J1 SM08B-SRSS-TB, U1 TLV76733DRVR, U12 INA186A3IDCKR, U18 LMR51420YDDCR, U5 XRIM160808SR47MBCD

Commit message: V-beta schematic in progress: buck/inductor/TVS/MOSFET swaps
Stan's V-beta edits via KiCad GUI:
- U13 LMR54406DBVR placed (replacing LMR51420)
- R119 = 115k for 10V output (Vfb=0.8V)
- U5 inductor value updated to FTC160808S4R7MBCA (4.7uH)
- D1 SMF24A-T13 TVS placed across +BATT/GND
- 24x SP40N03GNJ -> DOY180N03T (TDFN3333-8PL)
- 14x bulk caps in 1206 (replacing the 0805 swarm)
- R74 = 10R 0201 added between VDD and VDDA (no ferrite)
- Ferrites FB1-4 removed
- LMR54406 footprint and 3D imported via easyeda2kicad
- SMF24A-T13 footprint and 3D imported via easyeda2kicad

Schematic still has hygiene issues (footprint namespace prefixes,
cap/resistor R/C footprint swaps) to fix in a follow-up.

Generator version bumped to KiCad 10.0 (was 9.x).

Co-Authored-By: Claude Opus 4.7 (1M context) <noreply@anthropic.com>
Parts:
- removed C10, C11, C12, C13, C14, C15, C16, C17, C18, C19, C2, C20, C21, C22, C23, C24, C25, C26, C27, C28, C29, C3, C31, C4, C40, C41, C47, C5, C51, C6, C7, C8, C9: 10uF, Capacitor_SMD:C_0805_2012Metric, symbol Device:C
- removed U18: LMR51420YDDCR, components:SOT-23-6_L2.9-W1.6-P0.95-LS2.9-BL, symbol components:LMR51420YDDCR
- added CL32, CL33, CL34, CL35, CL36, CL37, CL38, CL39, CL40, CL41, CL42, CL43, CL45, CL46: 10uF, Capacitor_SMD:C_1206_3216Metric, symbol Device:C
- added D1: SMF24A-T13, 4in1ESC:SOD-123FL_L2.7-W1.8-LS3.7-RD, symbol components:SMF24A-T13
- added U13: LMR54406DBVR, 4in1ESC:SOT-23-6_L2.9-W1.6-P0.95-LS2.8-BR, symbol components:LMR54406DBVR
- R118, R73: footprint Capacitor_SMD:C_0201_0603Metric -> 4in1ESC:R_0201_0603Metric
- R119: value 124k -> 115k; LCSC C423759 -> C166341
- U5: value XRIM160808SR47MBCD -> FTC160808S4R7MBCA; LCSC C48391583 -> C46594347
Connections:
- net +BATT: now also CL32.1, CL33.1, CL34.1, CL35.1, CL36.1, CL37.1, CL38.1, CL39.1, CL40.1, CL41.1, CL42.1, CL43.1, CL45.1, CL46.1, D1.1 (K), U13.4 (EN), U13.5 (VIN)
- net GND: now also CL32.2, CL33.2, CL34.2, CL35.2, CL36.2, CL37.2, CL38.2, CL39.2, CL40.2, CL41.2, CL42.2, CL43.2, CL45.2, CL46.2, D1.2 (A), U13.2 (GND)
- net at R118.1, R119.2: now also U13.3 (FB)
- net at C72.1, U5.1: now also U13.6 (SW)
- net at C72.2: now also U13.1 (CB)
- net +8V renamed +10V
Other:
- moved on the sheet: C72

Commit message: V-beta hygiene: footprint namespace cleanup, R/C footprint swaps
Surgical line-by-line property-value substitutions (no structural
changes; paren balance and newline count preserved as sanity checks).

Changes (22 total):
- Inductor U5 footprint: components: -> 4in1ESC: (top sheet, 2 occurrences:
  lib_symbols cache + instance)
- NSG2065Q footprint: components: -> 4in1ESC:
- AT32F421 footprint: ESCLibrary: -> 4in1ESC:
- 17x resistor instances using Capacitor_SMD:C_0201_0603Metric
  swapped to Resistor_SMD:R_0201_0603Metric (ESC subsheet)

scripts/v_beta_hygiene_fix.py: dry-run / --apply mode, byte-level
operation in binary mode to avoid encoding mangles, paren-balance
and newline-count sanity checks before write.

Remaining cleanup (Stan, GUI): orphan placeholder symbols
(Reference="C","R" with ESCLibrary: lib_id) - delete by hand.
ESCLibrary: lib_id references on instances are still present
but resolve via the embedded lib_symbols cache.

Co-Authored-By: Claude Opus 4.7 (1M context) <noreply@anthropic.com>
Parts:
- U5: footprint components:IND-SMD_L1.6-W0.8_FTC160865SR47MBCA -> 4in1ESC:IND-SMD_L1.6-W0.8_FTC160865SR47MBCA
Changed lines of the file:
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@@
 			)
 		)
-		(property "Footprint" "components:IND-SMD_L1.6-W0.8_FTC160865SR47MBCA"
+		(property "Footprint" "4in1ESC:IND-SMD_L1.6-W0.8_FTC160865SR47MBCA"
 			(at 85.09 180.34 0)
 			(hide yes)
