File: 4in1ESC.kicad_sch (KiCad schematic)
At the start: 35 parts, among them J1 SM08B-SRSS-TB, U1 TLV76733DRVR, U12 INA186A3IDCKR, U13 LMR54406DBVR, U5 FTC160808S4R7MBCA

Commit message: alpha routing
Parts:
- removed CL33, CL34, CL35, CL36, CL37, CL38, CL39, CL40, CL41, CL42, CL43, CL45, CL46: 10uF, Capacitor_SMD:C_1206_3216Metric, symbol Device:C
- added D2: SMF24A-T13, 4in1ESC:SOD-123FL_L2.7-W1.8-LS3.7-RD, symbol components:SMF24A-T13
- R119: LCSC C166341 -> C166378
Connections:
- net +BATT: now also D2.1 (K)
- net GND: now also D2.2 (A)
Other:
- moved on the sheet: D1
