File: ESC.kicad_sch (KiCad schematic)
At the start: 36 parts, among them Q1 SP40N03GNJ, Q2 SP40N03GNJ, Q3 SP40N03GNJ, Q4 SP40N03GNJ, Q5 SP40N03GNJ, Q6 SP40N03GNJ, U2 AT32F421G8U7, U3 NSG2065Q

Commit message: V-beta schematic in progress: buck/inductor/TVS/MOSFET swaps
Stan's V-beta edits via KiCad GUI:
- U13 LMR54406DBVR placed (replacing LMR51420)
- R119 = 115k for 10V output (Vfb=0.8V)
- U5 inductor value updated to FTC160808S4R7MBCA (4.7uH)
- D1 SMF24A-T13 TVS placed across +BATT/GND
- 24x SP40N03GNJ -> DOY180N03T (TDFN3333-8PL)
- 14x bulk caps in 1206 (replacing the 0805 swarm)
- R74 = 10R 0201 added between VDD and VDDA (no ferrite)
- Ferrites FB1-4 removed
- LMR54406 footprint and 3D imported via easyeda2kicad
- SMF24A-T13 footprint and 3D imported via easyeda2kicad

Schematic still has hygiene issues (footprint namespace prefixes,
cap/resistor R/C footprint swaps) to fix in a follow-up.

Generator version bumped to KiCad 10.0 (was 9.x).

Co-Authored-By: Claude Opus 4.7 (1M context) <noreply@anthropic.com>
Parts:
- removed FB2: BLM03HD331SN1D, Inductor_SMD:L_0201_0603Metric, symbol Device:FerriteBead_Small
- added R74: 10R, Resistor_SMD:R_0201_0603Metric, symbol Device:R
- Q1, Q2, Q3, Q4, Q5, Q6: value SP40N03GNJ -> DOY180N03T; footprint components:POWERPAK-1212-8_L3.0-W3.0-P0.65-LS3.3-BL -> Package_SON:Diodes_PowerDI3333-8; LCSC C22466709 -> C49441966
Connections:
- net +3V3: now also R74.2; no longer C48.1
- net vdda: now reaches U2.5 (VDDA)
- net vdda: now also C48.1, R74.1
- net +8V renamed +10V
Other:
- moved on the sheet: C48, C49

Commit message: V-beta hygiene: footprint namespace cleanup, R/C footprint swaps
Surgical line-by-line property-value substitutions (no structural
changes; paren balance and newline count preserved as sanity checks).

Changes (22 total):
- Inductor U5 footprint: components: -> 4in1ESC: (top sheet, 2 occurrences:
  lib_symbols cache + instance)
- NSG2065Q footprint: components: -> 4in1ESC:
- AT32F421 footprint: ESCLibrary: -> 4in1ESC:
- 17x resistor instances using Capacitor_SMD:C_0201_0603Metric
  swapped to Resistor_SMD:R_0201_0603Metric (ESC subsheet)

scripts/v_beta_hygiene_fix.py: dry-run / --apply mode, byte-level
operation in binary mode to avoid encoding mangles, paren-balance
and newline-count sanity checks before write.

Remaining cleanup (Stan, GUI): orphan placeholder symbols
(Reference="C","R" with ESCLibrary: lib_id) - delete by hand.
ESCLibrary: lib_id references on instances are still present
but resolve via the embedded lib_symbols cache.

Co-Authored-By: Claude Opus 4.7 (1M context) <noreply@anthropic.com>
Parts:
- R16, R17, R18, R19, R21, R22, R23, R24, R25, R26, R27, R28, R29, R30, R31, R32, R33: footprint Capacitor_SMD:C_0201_0603Metric -> Resistor_SMD:R_0201_0603Metric
- U2: footprint ESCLibrary:QFN-28_L4.0-W4.0-P0.40-TL-EP2.4 -> 4in1ESC:QFN-28_L4.0-W4.0-P0.40-TL-EP2.4
- U3: footprint components:QFN-24_L4.0-W4.0-P0.50-TL-EP2.8 -> 4in1ESC:QFN-24_L4.0-W4.0-P0.50-TL-EP2.8
Changed lines of the file:
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@@
 			)
 		)
-		(property "Footprint" "Capacitor_SMD:C_0201_0603Metric"
+		(property "Footprint" "Resistor_SMD:R_0201_0603Metric"
 			(at 234.95 88.9 0)
 			(hide yes)
@@
 			)
 		)
-		(property "Footprint" "Capacitor_SMD:C_0201_0603Metric"
+		(property "Footprint" "Resistor_SMD:R_0201_0603Metric"
 			(at 240.03 111.76 0)
 			(hide yes)
@@
 			)
 		)
-		(property "Footprint" "Capacitor_SMD:C_0201_0603Metric"
+		(property "Footprint" "Resistor_SMD:R_0201_0603Metric"
 			(at 40.64 147.32 0)
 			(hide yes)
@@
 			)
 		)
-		(property "Footprint" "components:QFN-24_L4.0-W4.0-P0.50-TL-EP2.8"
+		(property "Footprint" "4in1ESC:QFN-24_L4.0-W4.0-P0.50-TL-EP2.8"
 			(at 133.35 85.09 0)
 			(hide yes)
@@
 			)
 		)
-		(property "Footprint" "Capacitor_SMD:C_0201_0603Metric"
+		(property "Footprint" "Resistor_SMD:R_0201_0603Metric"
 			(at 215.9 90.17 0)
 			(hide yes)
@@
 			)
 		)
-		(property "Footprint" "Capacitor_SMD:C_0201_0603Metric"
+		(property "Footprint" "Resistor_SMD:R_0201_0603Metric"
 			(at 210.82 88.9 0)
 			(hide yes)
@@
 			)
 		)
-		(property "Footprint" "Capacitor_SMD:C_0201_0603Metric"
+		(property "Footprint" "Resistor_SMD:R_0201_0603Metric"
 			(at 49.53 50.8 0)
 			(hide yes)
@@
 			)
 		)
-		(property "Footprint" "Capacitor_SMD:C_0201_0603Metric"
+		(property "Footprint" "Resistor_SMD:R_0201_0603Metric"
 			(at 259.08 88.9 0)
 			(hide yes)
@@
 			)
 		)
-		(property "Footprint" "Capacitor_SMD:C_0201_0603Metric"
+		(property "Footprint" "Resistor_SMD:R_0201_0603Metric"
 			(at 215.9 111.76 0)
 			(hide yes)
@@
 			)
 		)
-		(property "Footprint" "Capacitor_SMD:C_0201_0603Metric"
+		(property "Footprint" "Resistor_SMD:R_0201_0603Metric"
 			(at 243.84 90.17 0)
 			(hide yes)
@@
 			)
 		)
-		(property "Footprint" "Capacitor_SMD:C_0201_0603Metric"
+		(property "Footprint" "Resistor_SMD:R_0201_0603Metric"
 			(at 219.71 90.17 0)
 			(hide yes)
@@
 			)
 		)
-		(property "Footprint" "Capacitor_SMD:C_0201_0603Metric"
+		(property "Footprint" "Resistor_SMD:R_0201_0603Metric"
 			(at 100.33 162.56 0)
 			(hide yes)
@@
 			)
 		)
-		(property "Footprint" "ESCLibrary:QFN-28_L4.0-W4.0-P0.40-TL-EP2.4"
+		(property "Footprint" "4in1ESC:QFN-28_L4.0-W4.0-P0.40-TL-EP2.4"
 			(at 72.39 80.01 0)
 			(hide yes)
@@
 			)
 		)
-		(property "Footprint" "Capacitor_SMD:C_0201_0603Metric"
+		(property "Footprint" "Resistor_SMD:R_0201_0603Metric"
 			(at 161.29 161.29 0)
 			(hide yes)
@@
 			)
 		)
-		(property "Footprint" "Capacitor_SMD:C_0201_0603Metric"
+		(property "Footprint" "Resistor_SMD:R_0201_0603Metric"
 			(at 161.29 146.05 0)
 			(hide yes)
@@
 			)
 		)
-		(property "Footprint" "Capacitor_SMD:C_0201_0603Metric"
+		(property "Footprint" "Resistor_SMD:R_0201_0603Metric"
 			(at 100.33 147.32 0)
 			(hide yes)
@@
 			)
 		)
-		(property "Footprint" "Capacitor_SMD:C_0201_0603Metric"
+		(property "Footprint" "Resistor_SMD:R_0201_0603Metric"
 			(at 264.16 111.76 0)
 			(hide yes)
@@
 			)
 		)
-		(property "Footprint" "Capacitor_SMD:C_0201_0603Metric"
+		(property "Footprint" "Resistor_SMD:R_0201_0603Metric"
 			(at 40.64 162.56 0)
 			(hide yes)
@@
 			)
 		)
-		(property "Footprint" "Capacitor_SMD:C_0201_0603Metric"
+		(property "Footprint" "Resistor_SMD:R_0201_0603Metric"
 			(at 34.29 53.34 0)
 			(hide yes)
