File: 4in1-mini.kicad_pcb (KiCad board)
At the start: 6 copper layers, 31.2 x 33 mm, 186 parts, among them J1 SM08B-SRSS-TB, Q1 DOY180N03T, Q10 DOY180N03T, Q11 DOY180N03T, Q12 DOY180N03T, Q13 DOY180N03T, Q14 DOY180N03T, Q15 DOY180N03T, Q16 DOY180N03T, Q17 DOY180N03T, Q18 DOY180N03T, Q19 DOY180N03T, Q2 DOY180N03T, Q20 DOY180N03T, Q21 DOY180N03T, Q22 DOY180N03T, Q23 DOY180N03T, Q24 DOY180N03T, Q3 DOY180N03T, Q4 DOY180N03T, Q5 DOY180N03T, Q6 DOY180N03T, Q7 DOY180N03T, Q8 DOY180N03T, Q9 DOY180N03T, U1 TLV76733DRVR, U10 AT32F421G8U7, U11 NSG2065Q, U12 INA186A3IDCKR, U13 LMR54406DBVR, U2 AT32F421G8U7, U3 NSG2065Q, U5 FTC160808S4R7MBCA, U6 AT32F421G8U7, U7 NSG2065Q, U8 AT32F421G8U7, U9 NSG2065Q

Commit message: Routing update
Routing:
- net GND: vias 458 -> 457
Changed lines of the file:
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@@
 	)
 	(via
-		(at 86.282083 50.74425)
-		(size 0.35)
-		(drill 0.2)
-		(layers "F.Cu" "B.Cu")
-		(net "GND")
-	)
-	(via
 		(at 78.33 49.325)
 		(size 0.35)
@@
 		(polygon
 			(pts
-				(xy 71 61.25) (xy 71 59.5) (xy 73.75 58) (xy 75.75 58) (xy 75.75 60) (xy 72.5 61.25) (xy 70.9 61.25)
+				(xy 71 61.25) (xy 71 59.5) (xy 73.75 58) (xy 80.13 58) (xy 80.13 58.315385) (xy 72.5 61.25) (xy 70.9 61.25)
 			)
 		)
@@
 		(polygon
 			(pts
-				(xy 86.125 50.525) (xy 88.925 50.75) (xy 88.925 52.2) (xy 86.025 52.4)
+				(xy 86.36 50.88) (xy 88.925 50.75) (xy 88.925 52.2) (xy 86.025 52.4)
 			)
 		)
