File: 4in1-mini.kicad_sch (KiCad schematic)
At the start: 23 parts, among them J1 SM08B-SRSS-TB, U1 TLV76733DRVR, U12 INA186A3IDCKR, U13 LMR54406DBVR, U5 FTC160808S4R7MBCA

Commit message: meta: standardize symbol BOM/doc fields (20x20)
Add MPN/Manufacturer/LCSC/Digi-Key/Mouser/Farnell/Cost to every sourced
part. Source MPN + LCSC unit cost via keyless LCSC; Manufacturer set for
known ICs (TI, ArteryTek, Littelfuse). Clear legacy LCSC_Part, strip CJK
from Manufacturer. SMF24A-T13/DOY180N03T not in LCSC search -> MPN kept,
Cost blank. Digi-Key/Mouser/Farnell left blank pending API creds.
Properties-only -- no connectivity change. Also carries the finalized
on-canvas design comments.

Co-Authored-By: Claude Opus 4.8 (1M context) <noreply@anthropic.com>
Parts:
- C1, C42: Cost (none) -> 0.037; MPN (none) -> CL05A226MQ5QUNC
- C43, C86: Cost (none) -> 0.04157; MPN (none) -> CL10A226MO7JZNC
- C69, C70, C71, C72, C93, C94: Cost (none) -> 0.008457; MPN (none) -> GRM033R6YA104KE14D
- CL32: Cost (none) -> 0.05129; MPN (none) -> CL31B106KBHNNNE
- D1, D2: LCSC (none) -> C1977154; Manufacturer Littelfuse(美国力特) -> Littelfuse
- J1: Cost (none) -> 0.2523; MPN (none) -> SM08B-SRSS-TB(LF)(SN)
- R118: Cost (none) -> 0.0007714; MPN (none) -> RC0201FR-0710KL
- R119: Cost (none) -> 0.0005429; MPN (none) -> RTT011153FTH
- R73: Cost (none) -> 0.0006; MPN (none) -> 0201WMF1001TEE
- Rsense1: Cost (none) -> 0.2657; MPN (none) -> ASR-S-3-0.2F
- U1: Cost (none) -> 0.242; MPN (none) -> TLV76733DRVR; Manufacturer (none) -> Texas Instruments
- U12: Cost (none) -> 0.79; MPN (none) -> INA186A3IDCKR; Manufacturer (none) -> Texas Instruments
- U13: Cost (none) -> 0.4229; LCSC (none) -> C5219316; Manufacturer TI(德州仪器) -> Texas Instruments
- U5: Cost (none) -> 0.1079; MPN (none) -> FTC160808S4R7MBCA
Other:
- note added: "06/06/2026"
- note added: "2"
- note added: "4 to 36V, can handle 50V spikes. TBD on 8S 1.1Mhz, 0.6A (plenty for gate driving)"
- note added: "No telemetry signal pin, handled by Extended DSHOT protocol"
- note added: "Overview of OpenESC"
- note added: "SMFJ24A means there will be some leakage at fully charged 6S (25.2V) but voltage clamping gets improved too, will monitor this tradeoff"
- note added: "Total array of 20 decoupling caps At 25V DC Bias, only 1.5uF - 2uF derated per cap, so 30 - 40uF but very low ESR"
- moved on the sheet: C1, C42, C43, C69, C70, C71, C72, C86, CL32, D1, D2, R118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
